File: Lec Assignment 2/Changing Tone using Potentiometer/Changing Tone using Potentiometer.brd (EAGLE design)
At the start: 68.6 x 53.3 mm, 8 parts

Commit message: Lec Asg 2
Parts:
- removed D1, D2, D3: (no value), AUTODESK_CIRCUITS_BREADBOARD:LED5MM
- removed R1, R2, R3: 0.2k‎Ω, AUTODESK_CIRCUITS_BREADBOARD:0207/10
- added Rpot1: 250k‎Ω, AUTODESK_CIRCUITS_BREADBOARD:B25V
- moved PIEZO1 12.7 mm to (5.00, 35.5)
- renumbered U3 to U1
Connections:
- removed net N$6: R2.1, U1.5
- removed net N$7: D3.A, R3.2
- removed net N$8: R3.1, U1.4
- net N$1: now also Rpot1.E, U1.5V; no longer D1.K, D2.K, D3.K, PIEZO1.P$1, U1.GND
- net N$2: now also Rpot1.A, U1.GND.; no longer PIEZO1.P$2, U1.2
- net N$3: now also Rpot1.S, U1.A0; no longer D1.A, R1.2
- net N$4: now also PIEZO1.P$1, U1.GND; no longer R1.1, U1.6
- net N$5: now also PIEZO1.P$2, U1.8; no longer D2.A, R2.2
Changed lines of the file:
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@@
 </autorouter>
 <elements>
-<element value="" name="U3" library="AUTODESK_CIRCUITS_BREADBOARD" package="ARDUINO_UNO" x="5" y="10.08"></element><element value="" name="PIEZO1" library="AUTODESK_CIRCUITS_BREADBOARD" package="PIEZO-22MM" x="5" y="22.78"></element><element value="" name="D1" library="AUTODESK_CIRCUITS_BREADBOARD" package="LED5MM" x="5" y="35.480000000000004"></element><element value="" name="D2" library="AUTODESK_CIRCUITS_BREADBOARD" package="LED5MM" x="5" y="48.18"></element><element value="" name="D3" library="AUTODESK_CIRCUITS_BREADBOARD" package="LED5MM" x="5" y="60.879999999999995"></element><element value="0.2k‎Ω" name="R1" library="AUTODESK_CIRCUITS_BREADBOARD" package="0207/10" x="5" y="73.58"></element><element value="0.2k‎Ω" name="R2" library="AUTODESK_CIRCUITS_BREADBOARD" package="0207/10" x="5" y="86.28"></element><element value="0.2k‎Ω" name="R3" library="AUTODESK_CIRCUITS_BREADBOARD" package="0207/10" x="5" y="98.98"></element></elements>
+<element value="" name="U1" library="AUTODESK_CIRCUITS_BREADBOARD" package="ARDUINO_UNO" x="5" y="10.08"></element><element value="250k‎Ω" name="Rpot1" library="AUTODESK_CIRCUITS_BREADBOARD" package="B25V" x="5" y="22.78"></element><element value="" name="PIEZO1" library="AUTODESK_CIRCUITS_BREADBOARD" package="PIEZO-22MM" x="5" y="35.480000000000004"></element></elements>
 <signals>
-<signal name="N$1"><contactref element="PIEZO1" pad="P$1"></contactref><contactref element="U3" pad="GND"></contactref><wire x1="0" y1="22.78" x2="31.416" y2="60.879999999999995" width="0" layer="19" extent="1-1"></wire><contactref element="D1" pad="K"></contactref><wire x1="31.416" y1="60.879999999999995" x2="6.27" y2="35.480000000000004" width="0" layer="19" extent="1-1"></wire><contactref element="D2" pad="K"></contactref><wire x1="6.27" y1="35.480000000000004" x2="6.27" y2="48.18" width="0" layer="19" extent="1-1"></wire><contactref element="D3" pad="K"></contactref><wire x1="6.27" y1="48.18" x2="6.27" y2="60.879999999999995" width="0" layer="19" extent="1-1"></wire></signal><signal name="N$2"><contactref element="PIEZO1" pad="P$2"></contactref><contactref element="U3" pad="2"></contactref><wire x1="10" y1="22.78" x2="63.42" y2="60.879999999999995" width="0" layer="19" extent="1-1"></wire></signal><signal name="N$3"><contactref element="R1" pad="2"></contactref><contactref element="D1" pad="A"></contactref><wire x1="10.08" y1="73.58" x2="3.73" y2="35.480000000000004" width="0" layer="19" extent="1-1"></wire></signal><signal name="N$4"><contactref element="R1" pad="1"></contactref><contactref element="U3" pad="6"></contactref><wire x1="-0.08000000000000007" y1="73.58" x2="53.26" y2="60.879999999999995" width="0" layer="19" extent="1-1"></wire></signal><signal name="N$5"><contactref element="R2" pad="2"></contactref><contactref element="D2" pad="A"></contactref><wire x1="10.08" y1="86.28" x2="3.73" y2="48.18" width="0" layer="19" extent="1-1"></wire></signal><signal name="N$6"><contactref element="R2" pad="1"></contactref><contactref element="U3" pad="5"></contactref><wire x1="-0.08000000000000007" y1="86.28" x2="55.8" y2="60.879999999999995" width="0" layer="19" extent="1-1"></wire></signal><signal name="N$7"><contactref element="R3" pad="2"></contactref><contactref element="D3" pad="A"></contactref><wire x1="10.08" y1="98.98" x2="3.73" y2="60.879999999999995" width="0" layer="19" extent="1-1"></wire></signal><signal name="N$8"><contactref element="R3" pad="1"></contactref><contactref element="U3" pad="4"></contactref><wire x1="-0.08000000000000007" y1="98.98" x2="58.34" y2="60.879999999999995" width="0" layer="19" extent="1-1"></wire></signal></signals>
+<signal name="N$1"><contactref element="Rpot1" pad="E"></contactref><contactref element="U1" pad="5V"></contactref><wire x1="2.46" y1="23.415000000000003" x2="43.1" y2="12.620000000000001" width="0" layer="19" extent="1-1"></wire></signal><signal name="N$2"><contactref element="U1" pad="GND."></contactref><contactref element="Rpot1" pad="A"></contactref><wire x1="48.18" y1="12.620000000000001" x2="7.54" y2="23.415000000000003" width="0" layer="19" extent="1-1"></wire></signal><signal name="N$3"><contactref element="Rpot1" pad="S"></contactref><contactref element="U1" pad="A0"></contactref><wire x1="5" y1="23.415000000000003" x2="55.8" y2="12.620000000000001" width="0" layer="19" extent="1-1"></wire></signal><signal name="N$4"><contactref element="PIEZO1" pad="P$1"></contactref><contactref element="U1" pad="GND"></contactref><wire x1="0" y1="35.480000000000004" x2="31.416" y2="60.879999999999995" width="0" layer="19" extent="1-1"></wire></signal><signal name="N$5"><contactref element="PIEZO1" pad="P$2"></contactref><contactref element="U1" pad="8"></contactref><wire x1="10" y1="35.480000000000004" x2="46.656" y2="60.879999999999995" width="0" layer="19" extent="1-1"></wire></signal></signals>
 </board>
 </drawing>
